Commit message: Modified IK codes

File: skywalker/description/urdf/skywalker_model.xacro (robot description, xacro)
@@ -1,4 +1,4 @@
 <?xml version="1.0" ?>
-<robot xmlns:xacro="http://www.ros.org/wiki/xacro">
+<robot xmlns:xacro="http://ros.org/wiki/xacro" name="skywalker" >
 <!-- mir100-->
 <xacro:include filename="$(find mir_description)/urdf/include/mir_100_v1.urdf.xacro" />
@@ -39,5 +39,6 @@
     <parent link="box_link"/>
     <child link="ur5e_base_link"/>
-    <origin xyz="-0.3 0.1 0.245" rpy="0 0 0"/>
+    <!--origin xyz="-0.3 0.1 0.245" rpy="0 0 0"/-->
+        <origin xyz="-0.3 0.1 0.245" rpy="0 0 0"/>
   </joint>
 <!--joint name="ur5e_robotiq" type="fixed">

Commit message: Added Motion planning and optimization python codes

File: skywalker/description/urdf/skywalker_model.xacro (robot description, xacro)
@@ -17,5 +17,5 @@
 <!-- robotiq_2f_85_gripper -->
 <!--xacro:include filename="$(find robotiq_2f_85_gripper_visualization)/urdf/robotiq_arg2f_85_model_macro.xacro" />
-<xacro:robotiq_arg2f_85 prefix="gripper_"/-->
+<xacro:robotiq_arg2f_85 prefix=""/-->
 <!-- support -->
  <material name="blue">
@@ -39,10 +39,9 @@
     <parent link="box_link"/>
     <child link="ur5e_base_link"/>
-    <!--origin xyz="-0.3 0.1 0.245" rpy="0 0 0"/-->
-        <origin xyz="-0.3 0.1 0.245" rpy="0 0 0"/>
+    <origin xyz="-0.3 0.1 0.245" rpy="0 0 0"/>
   </joint>
 <!--joint name="ur5e_robotiq" type="fixed">
     <parent link="ur5e_tool0"/>
-    <child link="gripper_robotiq_arg2f_base_link"/>
+    <child link="robotiq_arg2f_base_link"/>
     <origin xyz="0 0 0" rpy="0 0 0"/>
   </joint-->
